Commit message: Updating the Robot URDF

File: src/abb_irb120/irb120_description/urdf/irb120.urdf (robot description, URDF)
Before this commit: robot abb_irb120, 29 links, 28 joints
Links:
- removed link BGA_1
- removed link BGA_10
- removed link BGA_11
- removed link BGA_12
- removed link BGA_13
- removed link BGA_14
- removed link BGA_15
- removed link BGA_16
- removed link BGA_2
- removed link BGA_3
- removed link BGA_4
- removed link BGA_5
- removed link BGA_6
- removed link BGA_7
- removed link BGA_8
- removed link BGA_9
- removed link PCB
- removed link Table
- removed link camera_frame
- removed link end_effector
- removed link end_frame
- removed link world
- added link base
- added link tool0
- link base_link: geometry collision mesh filename=package://abb_irb120_support/meshes/irb120_3_58/collision/b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; visual mesh filename=package://abb_irb120_support/meshes/irb120_3_58/visual/base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
- link link_1: geometry collision mesh filename=package://abb_irb120_support/meshes/irb120_3_58/collision/l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; visual mesh filename=package://abb_irb120_support/meshes/irb120_3_58/visual/link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
- link link_2: geometry collision mesh filename=package://abb_irb120_support/meshes/irb120_3_58/collision/l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; visual mesh filename=package://abb_irb120_support/meshes/irb120_3_58/visual/link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
- link link_3: geometry collision mesh filename=package://abb_irb120_support/meshes/irb120_3_58/collision/l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; visual mesh filename=package://abb_irb120_support/meshes/irb120_3_58/visual/link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
- link link_4: geometry collision mesh filename=package://abb_irb120_support/meshes/irb120_3_58/collision/l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; visual mesh filename=package://abb_irb120_support/meshes/irb120_3_58/visual/link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
- link link_5: geometry collision mesh filename=package://abb_irb120_support/meshes/irb120_3_58/collision/l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; visual mesh filename=package://abb_irb120_support/meshes/irb120_3_58/visual/link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
- link link_6: geometry collision mesh filename=package://abb_irb120_support/meshes/irb120_3_58/collision/l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; visual mesh filename=package://abb_irb120_support/meshes/irb120_3_58/visual/link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
Joints:
- removed joint PCB-BGA_1
- removed joint PCB-BGA_10
- removed joint PCB-BGA_11
- removed joint PCB-BGA_12
- removed joint PCB-BGA_13
- removed joint PCB-BGA_14
- removed joint PCB-BGA_15
- removed joint PCB-BGA_16
- removed joint PCB-BGA_2
- removed joint PCB-BGA_3
- removed joint PCB-BGA_4
- removed joint PCB-BGA_5
- removed joint PCB-BGA_6
- removed joint PCB-BGA_7
- removed joint PCB-BGA_8
- removed joint PCB-BGA_9
- removed joint Table-PCB
- removed joint base_link-Table
- removed joint end_effector-cameraframe
- removed joint end_effector-endframe
- removed joint fixed
- removed joint joint6-end_effector
- added joint base_link-base: type fixed, parent base_link, child base, origin xyz=0 0 0 rpy=0 0 0
- added joint joint6-tool0: type fixed, parent link_6, child tool0, origin xyz=0 0 0 rpy=0 0 0
- joint joint_1: limit lower=-2.87979 upper=2.87979 effort=20 velocity=4.36332 -> lower=-2.87979 upper=2.87979 effort=0 velocity=4.36332
- joint joint_2: limit lower=-1.91986 upper=1.91986 effort=20 velocity=4.36332 -> lower=-1.91986 upper=1.91986 effort=0 velocity=4.36332
- joint joint_3: limit lower=-1.91986 upper=1.22173 effort=20 velocity=4.36332 -> lower=-1.91986 upper=1.22173 effort=0 velocity=4.36332
- joint joint_4: limit lower=-2.79253 upper=2.79253 effort=20 velocity=5.58505 -> lower=-2.79253 upper=2.79253 effort=0 velocity=5.58505
- joint joint_5: limit lower=-2.094395 upper=2.094395 effort=20 velocity=5.58505 -> lower=-2.094395 upper=2.094395 effort=0 velocity=5.58505
- joint joint_6: limit lower=-6.98132 upper=6.98132 effort=20 velocity=7.33038 -> lower=-6.98132 upper=6.98132 effort=0 velocity=7.33038

File: src/abb_irb120/irb120_description/urdf/irb120.xacro (robot description, xacro)
@@ -228,11 +228,11 @@
   </link>
   <!-- joint - 6 ___ end_effector -->
-  <joint name="${prefix}joint6-end_effector" type="fixed">
+ <!--  <joint name="${prefix}joint6-end_effector" type="fixed">
   <parent link="${prefix}link_6"/>
   <child link="${prefix}end_effector"/>
   <origin rpy="0 0 0" xyz="0 0 0"/>
   </joint>
-<!--
- <link name="${prefix}end_effector">
+ -->
+ <!-- <link name="${prefix}end_effector">
  <inertial>
  <origin xyz="0 0 0" rpy="-1.57079632679 0 1.57079632679" />
@@ -256,7 +256,6 @@
  </geometry>
  </collision>
- </link>
--->
- <link name="${prefix}end_effector">
+ </link> -->
+ <!-- <link name="${prefix}end_effector">
   <visual>
    <origin xyz="0 0 0" rpy="-1.57079632679 0 1.57079632679" />
@@ -279,14 +278,14 @@
    <inertia ixx="1e-08" ixy="0" ixz="0" iyy="1e-08" iyz="0" izz="1e-08"/>
  </inertial>
- </link>
+ </link> -->
   <!-- end_effector ____ end_frame -->
-  <joint name="${prefix}vacuum_joint" type="revolute">
+ <!--  <joint name="${prefix}vacuum_joint" type="revolute">
   <parent link="${prefix}end_effector"/>
   <child link="${prefix}end_frame"/>
   <limit effort="30" velocity="1.0" lower="0" upper="0" />
   <origin rpy="0 0 0" xyz="0.160 0.0325 0"/>
-  </joint>
+  </joint> -->
   <!-- Description of end_frame -->
-  <link name="${prefix}end_frame">
+ <!--  <link name="${prefix}end_frame">
   <gravity>0</gravity>
   <inertial>
@@ -295,7 +294,7 @@
   <inertia ixx="1e-08" ixy="0" ixz="0" iyy="1e-08" iyz="0" izz="1e-08"/>
   </inertial>
-  </link>
+  </link> -->
  <gazebo>
- <plugin name="gazebo_ros_vacuum_gripper" filename="libgazebo_ros_vacuum_gripper.so">
+ <!-- <plugin name="gazebo_ros_vacuum_gripper" filename="libgazebo_ros_vacuum_gripper.so">
  <robotNamespace>irb120</robotNamespace>
  <bodyName>${prefix}end_frame</bodyName>
@@ -304,13 +303,13 @@
  <maxDistance>0.10</maxDistance>
  <minDistance>0.10</minDistance>
- </plugin>
+ </plugin> -->
  </gazebo>
- <joint name="${prefix}camera_joint" type="fixed">
+ <!-- <joint name="${prefix}camera_joint" type="fixed">
     <origin xyz="0.068 -0.0325 0" rpy="0 0 0"/>
     <parent link="${prefix}end_effector"/>
     <child link="${prefix}camera_link"/>
-  </joint>
+  </joint> -->
 <!-- Camera -->
-   <link name="${prefix}camera_link">
+   <!-- <link name="${prefix}camera_link">
    <collision>
    <origin xyz="0 0 0" rpy="1.57079632679 0 1.57079632679"/>
@@ -331,5 +330,5 @@
    <inertia ixx="1e-6" ixy="0" ixz="0" iyy="1e-6" iyz="0" izz="1e-6" />
    </inertial>
-   </link>
+   </link> -->
   <!-- end_effector ____ camera_frame -->
   <!--<joint name="${prefix}end_effector-cameraframe" type="fixed">
@@ -401,5 +400,5 @@
   </actuator>
   </transmission>
-  <transmission name="${prefix}tran7">
+  <!-- <transmission name="${prefix}tran7">
   <type>transmission_interface/SimpleTransmission</type>
   <joint name="${prefix}vacuum_joint">
@@ -410,5 +409,5 @@
   <mechanicalReduction>1</mechanicalReduction>
   </actuator>
-  </transmission>
+  </transmission> -->
 <!-- Gazebo-specific link properties -->
   <gazebo reference="${prefix}base_link">
@@ -441,10 +440,10 @@
   </gazebo>
  <!-- camera -->
-  <gazebo reference="${prefix}camera_link">
+  <!-- <gazebo reference="${prefix}camera_link">
     <sensor type="camera" name="camera1">
       <update_rate>30.0</update_rate>
       <camera name="head">
         <horizontal_fov>.95</horizontal_fov>
-        <!-- <horizontal_fov>0.95</horizontal_fov> -->
+        <!- <horizontal_fov>0.95</horizontal_fov> ->
         <image>
           <width>800</width>
@@ -458,7 +457,7 @@
         <noise>
           <type>gaussian</type>
-          <!-- Noise is sampled independently per pixel on each frame.
+          <!- Noise is sampled independently per pixel on each frame.
                That pixel's noise value is added to each of its color
-               channels, which at that point lie in the range [0,1]. -->
+               channels, which at that point lie in the range [0,1]. ->
           <mean>0.0</mean>
           <stddev>0.007</stddev>
@@ -480,5 +479,5 @@
       </plugin>
     </sensor>
-  </gazebo>
+  </gazebo> -->
 </xacro:macro>
 </robot>
